File: demo_project/demo_project.kicad_sch (KiCad schematic)
At the start: 22 parts, among them Q101 2N7000, SW101 LEFT, SW102 UP, SW103 RIGHT, SW104 DOWN

Commit message: blank sch starter
Parts:
- removed D102: YELLOW, LED_SMD:LED_0603_1608Metric_Pad1.05x0.95mm_HandSolder, symbol Device:LED
- removed D103: GREEN, LED_SMD:LED_0603_1608Metric_Pad1.05x0.95mm_HandSolder, symbol Device:LED
- removed D106: BLUE, LED_SMD:LED_0603_1608Metric_Pad1.05x0.95mm_HandSolder, symbol Device:LED
- removed LS101: Speaker, Buzzer_Beeper:MagneticBuzzer_ProjectsUnlimited_AI-4228-TWT-R, symbol Device:Speaker
- removed Q101: 2N7000, Package_TO_SOT_THT:TO-92_Inline, symbol Transistor_FET:2N7000
- removed VR101: RK09Y11L0001, footprints:alps_alpine_RK09Y11L0001, symbol alps_alpine_RK09Y11L0001:RK09Y11L0001
- added BT101: Battery, Battery:BatteryHolder_Keystone_2479_3xAAA, symbol Device:Battery
- added D104: WS2812B, LED_SMD:LED_WS2812B_PLCC4_5.0x5.0mm_P3.2mm, symbol LED:WS2812B
- added D105: GREEN, LED_THT:LED_D3.0mm_FlatTop, symbol Device:LED
- added J101: Conn_01x02, Connector_PinSocket_2.54mm:PinSocket_1x02_P2.54mm_Vertical, symbol Connector_Generic:Conn_01x02
- added J102: Conn_01x04, Connector_PinSocket_2.54mm:PinSocket_1x04_P2.54mm_Vertical, symbol Connector_Generic:Conn_01x04
- added SW105: SW_SPST, Connector:Banana_Jack_2Pin, symbol Switch:SW_SPST
- D101: footprint LED_SMD:LED_0603_1608Metric_Pad1.05x0.95mm_HandSolder -> LED_THT:LED_D3.0mm_FlatTop; Cost 0.0206 -> (none); Distributor JLCPCB -> (none); LCSC Part # C72038 -> (none); Manufacturer Everlight Elec -> (none); P/N 19-213/Y2C-CQ2R2L/3T(CY) -> (none)
- D102: renamed from D104; footprint LED_SMD:LED_0603_1608Metric_Pad1.05x0.95mm_HandSolder -> LED_THT:LED_D3.0mm_FlatTop; Cost 0.0248 -> (none); Distributor JLCPCB -> (none); LCSC Part # C72043 -> (none); Manufacturer Everlight Elec -> (none); P/N 19-217/GHC-YR1S2/3T -> (none)
- D103: renamed from D105; footprint LED_SMD:LED_0603_1608Metric_Pad1.05x0.95mm_HandSolder -> LED_THT:LED_D3.0mm_FlatTop; Cost 0.0169 -> (none); Distributor JLCPCB -> (none); LCSC Part # C72041 -> (none); Manufacturer Everlight Elec -> (none); P/N 19-217/BHC-ZL1M2RY/3T -> (none)
- R101, R102, R103, R104: footprint Resistor_SMD:R_1206_3216Metric_Pad1.30x1.75mm_HandSolder -> Resistor_THT:R_Axial_DIN0207_L6.3mm_D2.5mm_P10.16mm_Horizontal; Cost 0.0027 -> (none); Distributor JLCPCB -> (none); LCSC Part # C17902 -> (none); Manufacturer UNI-ROYAL -> (none); P/N 1206W4F1002T5E -> (none)
- SW101, SW102, SW103, SW104: Cost 0.0556 -> (none); Distributor JLCPCB -> (none); LCSC Part # C285474 -> (none); Manufacturer C&K -> (none); P/N PTS645SK432LFS -> (none)
Connections:
- net GND: no longer D101.1 (K), D102.1 (K), D103.1 (K)
- net VIN: now reaches A101.30 (VIN)
- net LED_BLUE: no longer names the net of A101.15 (D12)
- net LED_BLUE_PWM: no longer names the net of A101.12 (D9)
- net LED_BLUE_PWM: no longer D103.2 (A)
- net LED_GREEN: no longer names the net of A101.11 (D8)
- net LED_GREEN: no longer D102.2 (A)
- net LED_GREEN_PWM: no longer names the net of A101.14 (D11)
- net LED_YELLOW: no longer names the net of A101.10 (D7)
- net LED_YELLOW_PWM: no longer names the net of A101.13 (D10)
- net LED_YELLOW_PWM: no longer D101.2 (A)
- net POTENTIOMETER_AIN: no longer names the net of A101.19 (A0)
- net SPEAKER_PWM: no longer names the net of A101.9 (D6)
- no-connect marks 14 -> 21
Other:
- note added: "Battery footprint is 3xAAA (4.5 V)"
- note added: "Can also use a generic connector to hook up unmounted battery"
- note added: "Do not power w/ 5V USB at the same time."
- note added: "Power switch footprint is a banana plug (2pin) Feel free to replace with 1x2 generic 2.54mm pitch connector or your own."
- moved on the sheet: A101, D101, D102, D103, H101, H102, H103, H104, R101, R102, R103, R104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
